File: c64switchless_555.brd (EAGLE design)
At the start: 35.5 x 46.7 mm, 21 parts, among them IC1 7474N-RP, IC2 NE555, IC3 PIC12F629P, T1 BC547, T2 BC547, X1 B4B-ZR

Commit message: 555 based: updated R2,R3. Added revision.
Parts:
- R2, R3: value 100k -> 560k
Other:
- board text added: "Rev .1"
Changed lines of the file:
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@@
 <wire x1="35.54" y1="46.66" x2="0" y2="46.66" width="0" layer="20"/>
 <wire x1="0" y1="46.66" x2="0" y2="0" width="0" layer="20"/>
+<text x="16.51" y="44.45" size="1.778" layer="23">Rev .1</text>
 </plain>
 <attributes>
@@
 <element name="R1" library="rcl" package="0204/7" value="100k" x="5.08" y="5.08"/>
 <element name="T1" library="transistor" package="TO92" value="BC547" x="20.32" y="3.81"/>
-<element name="R2" library="rcl" package="0204/7" value="100k" x="27.94" y="36.83"/>
-<element name="R3" library="rcl" package="0204/7" value="100k" x="27.94" y="34.29"/>
+<element name="R2" library="rcl" package="0204/7" value="560k" x="27.94" y="36.83"/>
+<element name="R3" library="rcl" package="0204/7" value="560k" x="27.94" y="34.29"/>
 <element name="R4" library="rcl" package="0204/7" value="100k" x="12.7" y="13.97" rot="R180"/>
 <element name="C4" library="rcl" package="C050-030X075" value="100n" x="12.7" y="17.78" rot="R180"/>
